File: Hardware/Running_Hardware/Open_STMPLC_IO_V0.1/Open_STMPLC_IO_V0.1.kicad_pcb (KiCad board)
At the start: 2 copper layers, 207 x 120 mm, 593 parts, among them J1 Screw_Terminal_01x02, J10 Screw_Terminal_01x02, J11 Screw_Terminal_01x02, J12 Screw_Terminal_01x02, J13 Screw_Terminal_01x02, J14 Screw_Terminal_01x02, J15 Screw_Terminal_01x02, J16 Screw_Terminal_01x02, J17 Screw_Terminal_01x02, J18 Screw_Terminal_01x02, J19 Screw_Terminal_01x02, J2 Screw_Terminal_01x02, J20 Screw_Terminal_01x02, J21 Screw_Terminal_01x02, J22 Screw_Terminal_01x02, J23 Screw_Terminal_01x02, J24 Screw_Terminal_01x02, J25 Screw_Terminal_01x02, J26 Screw_Terminal_01x02, J27 Screw_Terminal_01x02, J28 Screw_Terminal_01x02, J29 Screw_Terminal_01x02, J3 Screw_Terminal_01x02, J30 Screw_Terminal_01x02, J31 Screw_Terminal_01x02, J32 Screw_Terminal_01x02, J33 Screw_Terminal_01x02, J34 Screw_Terminal_01x02, J35 Screw_Terminal_01x03, J36 Screw_Terminal_01x03, J37 Screw_Terminal_01x03, J38 Screw_Terminal_01x03, J39 10144517-041802LF, J4 Screw_Terminal_01x02, J40 Screw_Terminal_01x04, J41 10144517-041802LF, J42 10144517-041802LF, J43 Screw_Terminal_01x02, J5 Screw_Terminal_01x04, J6 Screw_Terminal_01x02, J7 Screw_Terminal_01x02, J8 Screw_Terminal_01x02, J9 Screw_Terminal_01x02, Q1 2N7002K, Q2 2N7002K, Q3 2N7002K, Q4 2N7002K, U1 TPS1H200A, U10 MAX31865xTP, U11 MAX31856, U12 6N137, U13 TPS1H200A, U14 TPS26600PWP, U15 NVTFS5124PLTAG, U16 TPS26600PWP, U17 NVTFS5124PLTAG, U18 TPS26600PWP, U19 NVTFS5124PLTAG, U2 TPS1H200A, U20 6N137, U21 6N137, U22 6N137, U23 6N137, U24 6N137, U25 6N137, U26 6N137, U27 6N137, U28 6N137, U29 6N137, U3 TPS1H200A, U30 6N137, U31 6N137, U32 6N137, U33 6N137, U34 6N137, U35 6N137, U36 6N137, U37 XTR305, U38 XTR305, U39 AD4111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

Commit message: Common GND terminal changes
Parts:
- removed C46, C47, C48, C49, C50, C51: 100nF, Capacitor_SMD:C_0603_1608Metric_Pad1.08x0.95mm_HandSolder
- removed D100, D101, D106, D107, D94, D95: NSI50010YT1G, Diode_SMD:D_SOD-123
- removed D102, D103, D90, D91, D96, D97: SMAJ33CA, Diode_SMD:D_SMA
- removed D104, D105, D92, D93, D98, D99: MB110S, Package_TO_SOT_SMD:TO-269AA
- removed D153, D154, D155, D156, D157, D158: LED, LED_SMD:LED_0603_1608Metric_Pad1.05x0.95mm_HandSolder
- removed J10, J11, J12, J13, J14, J15, J27, J28, J29, J30, J31, J32, J6, J7, J8, J9: Screw_Terminal_01x02, TerminalBlock_Phoenix:TerminalBlock_Phoenix_MKDS-1-2-3.81_1x02_P3.81mm_Horizontal
- removed R146, R147, R152, R153, R158, R159: 10R/1W, Resistor_SMD:R_0603_1608Metric_Pad0.98x0.95mm_HandSolder
- removed R148, R149, R154, R155, R160, R161: 2.2K, Resistor_SMD:R_0603_1608Metric_Pad0.98x0.95mm_HandSolder
- removed R150, R151, R156, R157, R162, R163, R239, R240, R241, R242, R243, R244: 1K, Resistor_SMD:R_0603_1608Metric_Pad0.98x0.95mm_HandSolder
- removed U31, U32, U33, U34, U35, U36: 6N137, Package_DIP:DIP-8_W7.62mm
- added C89: 470uF/50V, Capacitor_THT:CP_Radial_D10.0mm_P5.00mm, F.Cu at (47.8, 14.0)
- added F5: 0685T5000-01, Fuse:Fuse_1206_3216Metric, F.Cu at (58.9, 13.3)
- added FB4: BLM31SN500SH1L, Inductor_SMD:L_1206_3216Metric_Pad1.22x1.90mm_HandSolder, F.Cu at (59.2, 9.91)
- added Q5: AOD407, Package_TO_SOT_SMD:TO-252-3_TabPin2, F.Cu at (51.2, 4.17)
- added R245: 100K, Resistor_SMD:R_0603_1608Metric_Pad0.98x0.95mm_HandSolder, F.Cu at (58.3, 16.2)
- D159: value SS510 -> BZV55C10; footprint Diode_SMD:D_SMA -> Diode_SMD:D_MiniMELF
- J1: value Screw_Terminal_01x02 -> Screw_Terminal_01x10; footprint TerminalBlock_Phoenix:TerminalBlock_Phoenix_MKDS-1-2-3.81_1x02_P3.81mm_Horizontal -> TerminalBlock_Phoenix:TerminalBlock_Phoenix_MKDS-1-10-3.81_1x10_P3.81mm_Horizontal
- J2: value Screw_Terminal_01x02 -> Screw_Terminal_01x06; footprint TerminalBlock_Phoenix:TerminalBlock_Phoenix_MKDS-1-2-3.81_1x02_P3.81mm_Horizontal -> TerminalBlock_Phoenix:TerminalBlock_Phoenix_MKDS-1-6-3.81_1x06_P3.81mm_Horizontal
- moved J33 47.4 mm to (152.5, 144.0)
- moved J34 47.4 mm to (161.5, 144.0)
- moved J40 47.0 mm to (117.8, 35.5)
- moved J5 47.0 mm to (134.8, 35.5)
- moved J2 20.4 mm to (179.5, 144.0)
- moved J4 20.4 mm to (170.5, 144.0)
- moved J1 19.4 mm to (112.8, 144.0)
- moved J16 10.9 mm to (233.9, 35.5)
- moved J17 10.9 mm to (224.9, 35.5)
- moved J18 10.9 mm to (215.9, 35.5)
- moved J19 10.9 mm to (206.9, 35.5)
- moved J20 10.9 mm to (197.9, 35.5)
- moved J21 10.9 mm to (188.9, 35.5)
- moved J22 10.9 mm to (179.9, 35.5)
- moved J23 10.9 mm to (170.9, 35.5)
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Connections:
- D1 pad 1: Net-(D1-K) -> /B2B_Connector/DIG_HS_OUT_TERMINAL_1
- D13 pad 1: Net-(D13-K) -> /B2B_Connector/DIG_OUT_TERMINAL_2
- D14 pad 1: Net-(D13-K) -> /B2B_Connector/DIG_OUT_TERMINAL_2
- D159 pad 1: +24V -> Net-(D159-K)
- D160 pad 1: Net-(D159-A) -> Net-(D160-A1)
- D17 pad 1: Net-(D17-K) -> /B2B_Connector/DIG_OUT_TERMINAL_3
- D18 pad 1: Net-(D17-K) -> /B2B_Connector/DIG_OUT_TERMINAL_3
- D21 pad 1: Net-(D21-K) -> /B2B_Connector/DIG_OUT_TERMINAL_4
- D22 pad 1: Net-(D21-K) -> /B2B_Connector/DIG_OUT_TERMINAL_4
- D25 pad 1: Net-(D25-K) -> /B2B_Connector/DIG_OUT_TERMINAL_5
- D26 pad 1: Net-(D25-K) -> /B2B_Connector/DIG_OUT_TERMINAL_5
- D29 pad 1: Net-(D29-K) -> /B2B_Connector/DIG_OUT_TERMINAL_6
- D3 pad 1: Net-(D1-K) -> /B2B_Connector/DIG_HS_OUT_TERMINAL_1
- D30 pad 1: Net-(D29-K) -> /B2B_Connector/DIG_OUT_TERMINAL_6
- D37 pad 1: Net-(D37-K) -> /B2B_Connector/DIG_HS_OUT_TERMINAL_2
- D38 pad 1: Net-(D37-K) -> /B2B_Connector/DIG_HS_OUT_TERMINAL_2
- D42 pad 1: Net-(D42-K) -> /B2B_Connector/DIG_HS_OUT_TERMINAL_3
- D43 pad 1: Net-(D42-K) -> /B2B_Connector/DIG_HS_OUT_TERMINAL_3
- D47 pad 1: Net-(D47-K) -> /B2B_Connector/DIG_HS_OUT_TERMINAL_4
- D48 pad 1: Net-(D47-K) -> /B2B_Connector/DIG_HS_OUT_TERMINAL_4
- D5 pad 1: Net-(D5-A1) -> /B2B_Connector/DIG_OUT_TERMINAL_1
- D51 pad 1: Net-(D51-K) -> /B2B_Connector/DIG_OUT_TERMINAL_7
- D52 pad 1: Net-(D51-K) -> /B2B_Connector/DIG_OUT_TERMINAL_7
- D55 pad 1: Net-(D55-K) -> /B2B_Connector/DIG_OUT_TERMINAL_8
- D56 pad 1: Net-(D55-K) -> /B2B_Connector/DIG_OUT_TERMINAL_8
- D6 pad 1: Net-(D5-A1) -> /B2B_Connector/DIG_OUT_TERMINAL_1
- J1 pad 1: Net-(D1-K) -> GND
- J1 pad 2: GND -> /B2B_Connector/DIG_OUT_TERMINAL_8
- J2 pad 1: Net-(D5-A1) -> GND
- J2 pad 2: GND -> /B2B_Connector/DIG_HS_OUT_TERMINAL_4
- J43 pad 2: Net-(D159-A) -> Net-(J43-Pin_2)
- R215 pad 2: Net-(D1-K) -> /B2B_Connector/DIG_HS_OUT_TERMINAL_1
- R216 pad 2: Net-(D37-K) -> /B2B_Connector/DIG_HS_OUT_TERMINAL_2
- R217 pad 2: Net-(D42-K) -> /B2B_Connector/DIG_HS_OUT_TERMINAL_3
- R218 pad 2: Net-(D47-K) -> /B2B_Connector/DIG_HS_OUT_TERMINAL_4
- R219 pad 2: Net-(D5-A1) -> /B2B_Connector/DIG_OUT_TERMINAL_1
- R220 pad 2: Net-(D13-K) -> /B2B_Connector/DIG_OUT_TERMINAL_2
- R221 pad 2: Net-(D17-K) -> /B2B_Connector/DIG_OUT_TERMINAL_3
- R222 pad 2: Net-(D21-K) -> /B2B_Connector/DIG_OUT_TERMINAL_4
- R223 pad 2: Net-(D25-K) -> /B2B_Connector/DIG_OUT_TERMINAL_5
- R224 pad 2: Net-(D29-K) -> /B2B_Connector/DIG_OUT_TERMINAL_6
- R225 pad 2: Net-(D51-K) -> /B2B_Connector/DIG_OUT_TERMINAL_7
- R226 pad 2: unconnected-(R226-Pad2) -> /B2B_Connector/DIG_OUT_TERMINAL_8

Commit message: Rule areas creation
Parts:
- removed J16, J17, J18, J19, J20, J21, J22, J23, J24, J25, J26: Screw_Terminal_01x02, TerminalBlock_Phoenix:TerminalBlock_Phoenix_MKDS-1-2-3.81_1x02_P3.81mm_Horizontal
- added J6: Screw_Terminal_01x04, TerminalBlock_Phoenix:TerminalBlock_Phoenix_MKDS-1-4-3.81_1x04_P3.81mm_Horizontal, F.Cu at (181.4, 35.5)
- added J7: Screw_Terminal_01x04, TerminalBlock_Phoenix:TerminalBlock_Phoenix_MKDS-1-4-3.81_1x04_P3.81mm_Horizontal, F.Cu at (197.9, 35.5)
- added J8: Screw_Terminal_01x04, TerminalBlock_Phoenix:TerminalBlock_Phoenix_MKDS-1-4-3.81_1x04_P3.81mm_Horizontal, F.Cu at (214.4, 35.5)
- J3: value Screw_Terminal_01x02 -> Screw_Terminal_01x04; footprint TerminalBlock_Phoenix:TerminalBlock_Phoenix_MKDS-1-2-3.81_1x02_P3.81mm_Horizontal -> TerminalBlock_Phoenix:TerminalBlock_Phoenix_MKDS-1-4-3.81_1x04_P3.81mm_Horizontal
- moved J4 111.9 mm to (142.5, 35.7), turned to 180 degrees
- moved J40 41.4 mm to (159.2, 35.6)
- moved J5 41.4 mm to (176.2, 35.6)
- moved J33 33.2 mm to (185.7, 144.0)
- moved J34 33.2 mm to (194.7, 144.0)
- moved J2 18.5 mm to (161.0, 143.9)
- moved J1 8.69 mm to (121.5, 144.0)
Connections:
- D11 pad 4: Net-(D8-A2) -> /DIG_IN_GRP2/COMC
- D57 pad 4: Net-(D9-A2) -> /DIG_IN_GRP2/COMD
- D60 pad 2: Net-(D60-A2) -> /DIG_IN_GRP2/COMC
- D61 pad 2: Net-(D61-A2) -> /DIG_IN_GRP2/COMD
- D62 pad 4: Net-(D60-A2) -> /DIG_IN_GRP2/COMC
- D63 pad 4: Net-(D61-A2) -> /DIG_IN_GRP2/COMD
- D66 pad 2: Net-(D66-A2) -> /DIG_IN_GRP2/COMC
- D67 pad 2: Net-(D67-A2) -> /DIG_IN_GRP2/COMD
- D68 pad 4: Net-(D66-A2) -> /DIG_IN_GRP2/COMC
- D69 pad 4: Net-(D67-A2) -> /DIG_IN_GRP2/COMD
- D72 pad 2: Net-(D72-A2) -> /DIG_IN_GRP1/COMA
- D73 pad 2: Net-(D73-A2) -> /DIG_IN_GRP1/COMB
- D74 pad 4: Net-(D72-A2) -> /DIG_IN_GRP1/COMA
- D75 pad 4: Net-(D73-A2) -> /DIG_IN_GRP1/COMB
- D78 pad 2: Net-(D78-A2) -> /DIG_IN_GRP1/COMA
- D79 pad 2: Net-(D79-A2) -> /DIG_IN_GRP1/COMB
- D8 pad 2: Net-(D8-A2) -> /DIG_IN_GRP2/COMC
- D80 pad 4: Net-(D78-A2) -> /DIG_IN_GRP1/COMA
- D81 pad 4: Net-(D79-A2) -> /DIG_IN_GRP1/COMB
- D84 pad 2: Net-(D84-A2) -> /DIG_IN_GRP1/COMA
- D85 pad 2: Net-(D85-A2) -> /DIG_IN_GRP1/COMB
- D86 pad 4: Net-(D84-A2) -> /DIG_IN_GRP1/COMA
- D87 pad 4: Net-(D85-A2) -> /DIG_IN_GRP1/COMB
- D9 pad 2: Net-(D9-A2) -> /DIG_IN_GRP2/COMD
- J3 pad 1: Net-(J3-Pin_1) -> /DIG_IN_GRP2/DIG_IN_TERMINAL_9
- J3 pad 2: Net-(D8-A2) -> /DIG_IN_GRP2/DIG_IN_TERMINAL_8
- R116 pad 1: Net-(J17-Pin_1) -> /DIG_IN_GRP2/DIG_IN_TERMINAL_8
- R117 pad 1: Net-(J18-Pin_1) -> /DIG_IN_GRP2/DIG_IN_TERMINAL_11
- R122 pad 1: Net-(J19-Pin_1) -> /DIG_IN_GRP2/DIG_IN_TERMINAL_9
- R123 pad 1: unconnected-(R123-Pad1) -> /DIG_IN_GRP2/DIG_IN_TERMINAL_12
- R128 pad 1: Net-(J21-Pin_1) -> /DIG_IN_GRP1/DIG_IN_TERMINAL_1
- R129 pad 1: Net-(J22-Pin_1) -> /DIG_IN_GRP1/DIG_IN_TERMINAL_4
- R134 pad 1: Net-(J23-Pin_1) -> /DIG_IN_GRP1/DIG_IN_TERMINAL_2
- R135 pad 1: Net-(J24-Pin_1) -> /DIG_IN_GRP1/DIG_IN_TERMINAL_5
- R140 pad 1: Net-(J25-Pin_1) -> /DIG_IN_GRP1/DIG_IN_TERMINAL_3
- R141 pad 1: unconnected-(R141-Pad1) -> /DIG_IN_GRP1/DIG_IN_TERMINAL_6
- R22 pad 1: Net-(J3-Pin_1) -> /DIG_IN_GRP2/DIG_IN_TERMINAL_7
- R25 pad 1: Net-(J16-Pin_1) -> /DIG_IN_GRP2/DIG_IN_TERMINAL_10

Commit message: IO board component grouping
Parts:
- added R146: 10R/1W, Resistor_SMD:R_2512_6332Metric_Pad1.40x3.35mm_HandSolder, F.Cu at (45.0, -84.5)
- added R147: 10R/1W, Resistor_SMD:R_2512_6332Metric_Pad1.40x3.35mm_HandSolder, F.Cu at (45.0, -82.0)
- added R148: 10R/1W, Resistor_SMD:R_2512_6332Metric_Pad1.40x3.35mm_HandSolder, F.Cu at (-25.0, -71.0)
- added R149: 10R/1W, Resistor_SMD:R_2512_6332Metric_Pad1.40x3.35mm_HandSolder, F.Cu at (45.0, -77.0)
- added R150: 10R/1W, Resistor_SMD:R_2512_6332Metric_Pad1.40x3.35mm_HandSolder, F.Cu at (45.0, -74.5)
- added R151: 10R/1W, Resistor_SMD:R_2512_6332Metric_Pad1.40x3.35mm_HandSolder, F.Cu at (45.0, -72.0)
- added R152: 10R/1W, Resistor_SMD:R_2512_6332Metric_Pad1.40x3.35mm_HandSolder, F.Cu at (122.0, -78.7)
- added R153: 10R/1W, Resistor_SMD:R_2512_6332Metric_Pad1.40x3.35mm_HandSolder, F.Cu at (122.0, -76.1)
- added R154: 10R/1W, Resistor_SMD:R_2512_6332Metric_Pad1.40x3.35mm_HandSolder, F.Cu at (122.0, -73.6)
- added R155: 10R/1W, Resistor_SMD:R_2512_6332Metric_Pad1.40x3.35mm_HandSolder, F.Cu at (122.0, -71.1)
- added R156: 10R/1W, Resistor_SMD:R_2512_6332Metric_Pad1.40x3.35mm_HandSolder, F.Cu at (122.0, -68.6)
- added R157: 10R/1W, Resistor_SMD:R_2512_6332Metric_Pad1.40x3.35mm_HandSolder, F.Cu at (122.0, -66.1)
- R116, R117, R122, R123, R128, R129, R134, R135, R140, R141, R22, R25: footprint Resistor_SMD:R_0603_1608Metric_Pad0.98x0.95mm_HandSolder -> Resistor_SMD:R_2512_6332Metric_Pad1.40x3.35mm_HandSolder
- moved C3 308.0 mm to (156.1, -68.4)
- moved C35 308.0 mm to (156.1, -65.9)
- moved C36 308.0 mm to (156.1, -63.4)
- moved C37 308.0 mm to (156.1, -60.9)
- moved C38 308.0 mm to (156.1, -58.4)
- moved C39 308.0 mm to (156.1, -55.8)
- moved D11 308.0 mm to (135.7, -66.5)
- moved D147 308.0 mm to (156.1, -48.3)
- moved D148 308.0 mm to (156.1, -45.7)
- moved D149 308.0 mm to (156.1, -43.1)
- moved D150 308.0 mm to (156.1, -40.5)
- moved D151 308.0 mm to (156.1, -37.9)
- moved D152 308.0 mm to (156.1, -35.3)
- moved D57 308.0 mm to (135.7, -60.1)
- moved D58 308.0 mm to (151.0, -68.0)
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Connections:
- D11 pad 4: /DIG_IN_GRP2/COMC -> Net-(D8-A2)
- D57 pad 4: /DIG_IN_GRP2/COMD -> Net-(D9-A2)
- D60 pad 2: /DIG_IN_GRP2/COMC -> Net-(D60-A2)
- D61 pad 2: /DIG_IN_GRP2/COMD -> Net-(D61-A2)
- D62 pad 4: /DIG_IN_GRP2/COMC -> Net-(D60-A2)
- D63 pad 4: /DIG_IN_GRP2/COMD -> Net-(D61-A2)
- D66 pad 2: /DIG_IN_GRP2/COMC -> Net-(D66-A2)
- D67 pad 2: /DIG_IN_GRP2/COMD -> Net-(D67-A2)
- D68 pad 4: /DIG_IN_GRP2/COMC -> Net-(D66-A2)
- D69 pad 4: /DIG_IN_GRP2/COMD -> Net-(D67-A2)
- D72 pad 2: /DIG_IN_GRP1/COMA -> Net-(D72-A2)
- D73 pad 2: /DIG_IN_GRP1/COMB -> Net-(D73-A2)
- D74 pad 4: /DIG_IN_GRP1/COMA -> Net-(D72-A2)
- D75 pad 4: /DIG_IN_GRP1/COMB -> Net-(D73-A2)
- D78 pad 2: /DIG_IN_GRP1/COMA -> Net-(D78-A2)
- D79 pad 2: /DIG_IN_GRP1/COMB -> Net-(D79-A2)
- D8 pad 2: /DIG_IN_GRP2/COMC -> Net-(D8-A2)
- D80 pad 4: /DIG_IN_GRP1/COMA -> Net-(D78-A2)
- D81 pad 4: /DIG_IN_GRP1/COMB -> Net-(D79-A2)
- D84 pad 2: /DIG_IN_GRP1/COMA -> Net-(D84-A2)
- D85 pad 2: /DIG_IN_GRP1/COMB -> Net-(D85-A2)
- D86 pad 4: /DIG_IN_GRP1/COMA -> Net-(D84-A2)
- D87 pad 4: /DIG_IN_GRP1/COMB -> Net-(D85-A2)
- D9 pad 2: /DIG_IN_GRP2/COMD -> Net-(D9-A2)

Commit message: IO board component placement
Parts:
- added H1: MountingHole, MountingHole:MountingHole_3.2mm_M3, F.Cu at (51.5, 74.0)
- added H2: MountingHole, MountingHole:MountingHole_3.2mm_M3, F.Cu at (51.5, 136.0)
- added H3: MountingHole, MountingHole:MountingHole_3.2mm_M3, F.Cu at (211.0, 62.0)
- added H4: MountingHole, MountingHole:MountingHole_3.2mm_M3, F.Cu at (213.5, 105.0)
- added H5: MountingHole, MountingHole:MountingHole_3.2mm_M3, F.Cu at (213.5, 148.0)
- U12, U20, U21, U22, U23, U24, U25, U26, U27, U28, U29, U30: footprint Package_DIP:DIP-8_W7.62mm -> Package_DIP:SMDIP-8_W9.53mm_Clearance8mm
- moved J41 270.3 mm to (212.5, 83.0), turned to 90 degrees
- moved J42 265.4 mm to (212.5, 127.5), turned to 90 degrees
- moved D35 238.6 mm to (69.0, 86.0), turned to 90 degrees
- moved R216 236.5 mm to (70.5, 74.5), turned to -90 degrees
- moved D38 236.2 mm to (63.5, 73.0), turned to 180 degrees
- moved D130 233.5 mm to (73.0, 74.5), turned to 90 degrees
- moved U14 232.9 mm to (63.5, 96.0)
- moved Q1 232.2 mm to (70.0, 81.0), turned to -90 degrees
- moved U15 230.5 mm to (62.5, 86.0), turned to -90 degrees
- moved D37 229.5 mm to (63.5, 77.0), turned to 180 degrees
- moved R88 228.9 mm to (70.0, 77.5)
- moved R90 228.7 mm to (66.5, 86.0), turned to -90 degrees
- moved R87 224.3 mm to (73.0, 78.5), turned to -90 degrees
- moved R89 223.5 mm to (71.5, 86.0), turned to -90 degrees
- moved R12 223.2 mm to (58.0, 93.5), turned to 90 degrees
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Routing:
- net +3V3: track 0.00 -> 122.2 mm
- net Net-(U7-MODE): track 0.00 -> 20.1 mm, vias 0 -> 1
- net Net-(U18-MODE): track 0.00 -> 20.1 mm, vias 0 -> 1
- net Net-(U16-MODE): track 0.00 -> 20.1 mm, vias 0 -> 1
- net Net-(U14-MODE): track 0.00 -> 20.1 mm, vias 0 -> 1
- net Net-(D44-K): track 0.00 -> 18.6 mm
- net Net-(D39-K): track 0.00 -> 18.5 mm
- net Net-(D33-K): track 0.00 -> 18.5 mm
- net Net-(D34-K): track 0.00 -> 18.5 mm
- net Net-(D15-K): track 0.00 -> 15.5 mm, vias 0 -> 2
- net Net-(D13-A): track 0.00 -> 15.5 mm, vias 0 -> 2
- net Net-(D31-K): track 0.00 -> 15.5 mm, vias 0 -> 2
- net Net-(D27-K): track 0.00 -> 15.5 mm, vias 0 -> 2
- net Net-(D23-K): track 0.00 -> 15.5 mm, vias 0 -> 2
- net Net-(D19-K): track 0.00 -> 15.5 mm, vias 0 -> 2
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Other:
- board size 207 x 120 mm -> 169 x 90 mm

Commit message: IO board layout
Parts:
- added C46: 10uF, Capacitor_SMD:C_0805_2012Metric_Pad1.18x1.45mm_HandSolder, F.Cu at (38.7, 37.5)
- added C47: 1uF, Capacitor_SMD:C_0603_1608Metric_Pad1.08x0.95mm_HandSolder, F.Cu at (34.2, 22.4)
- added C48: 100nF, Capacitor_SMD:C_0603_1608Metric_Pad1.08x0.95mm_HandSolder, F.Cu at (34.2, 24.9)
- added C50: 1uF, Capacitor_SMD:C_0603_1608Metric_Pad1.08x0.95mm_HandSolder, F.Cu at (34.2, 27.4)
- added C51: 1uF, Capacitor_SMD:C_0603_1608Metric_Pad1.08x0.95mm_HandSolder, F.Cu at (34.2, 29.9)
- added C90: 100nF, Capacitor_SMD:C_0603_1608Metric_Pad1.08x0.95mm_HandSolder, F.Cu at (34.2, 32.5)
- added D90: BZV55C10, Diode_SMD:D_MiniMELF, F.Cu at (39.6, 31.0)
- added D91: MMSZ5256ET1G, Diode_SMD:D_MiniMELF, F.Cu at (39.6, 34.4)
- added Q6: AOD407, Package_TO_SOT_SMD:TO-252-3_TabPin2, F.Cu at (43.3, 25.3)
- added Q7: MMBT5401, Package_TO_SOT_SMD:SOT-23, F.Cu at (45.2, 31.6)
- added R158: 100K, Resistor_SMD:R_0603_1608Metric_Pad0.98x0.95mm_HandSolder, F.Cu at (34.2, 35.0)
- added R159: 10K, Resistor_SMD:R_0603_1608Metric_Pad0.98x0.95mm_HandSolder, F.Cu at (34.2, 37.5)
- added R160: 10K, Resistor_SMD:R_0603_1608Metric_Pad0.98x0.95mm_HandSolder, F.Cu at (34.2, 40.0)
- added R161: 100K, Resistor_SMD:R_0603_1608Metric_Pad0.98x0.95mm_HandSolder, F.Cu at (34.2, 42.5)
- added R162: 100K, Resistor_SMD:R_0603_1608Metric_Pad0.98x0.95mm_HandSolder, F.Cu at (34.2, 45.0)
- C3, C35, C36, C37, C38, C39, C40, C41, C42, C43, C44, C45, D11, D141, D142, D143, D144, D145, D146, D147, D148, D149, D150, D151, D152, D57, D58, D59, D60, D61, D62, D63, D64, D65, D66, D67, D68, D69, D70, D71, D72, D73, D74, D75, D76, D77, D78, D79, D8, D80, D81, D82, D83, D84, D85, D86, D87, D88, D89, D9, R113, R114, R115, R116, R117, R118, R119, R120, R121, R122, R123, R124, R125, R126, R127, R128, R129, R130, R131, R132, R133, R134, R135, R136, R137, R138, R139, R140, R141, R142, R143, R144, R145, R146, R147, R148, R149, R150, R151, R152, R153, R154, R155, R156, R157, R22, R227, R228, R229, R230, R231, R232, R233, R234, R235, R236, R237, R238, R25, R27, U12, U20, U21, U22, U23, U24, U25, U26, U27, U28, U29, U30: moved to B.Cu
- moved D119 339.9 mm to (204.2, 134.5), turned to 180 degrees
- moved C71 336.3 mm to (205.5, 129.0)
- moved F1 335.1 mm to (205.5, 138.5), turned to 180 degrees
- moved D118 334.6 mm to (199.2, 138.5), turned to 180 degrees
- moved C70 332.0 mm to (201.5, 129.0), turned to 180 degrees
- moved C69 327.7 mm to (197.5, 131.0), turned to 180 degrees
- moved D122 327.6 mm to (190.9, 134.5), turned to 180 degrees
- moved R192 323.4 mm to (201.5, 131.0)
- moved D124 323.1 mm to (185.9, 138.5), turned to 180 degrees
- moved F3 322.6 mm to (192.2, 138.5), turned to 180 degrees
- moved R194 322.0 mm to (205.5, 131.0), turned to 180 degrees
- moved C67 318.5 mm to (186.2, 107.5), turned to 90 degrees
- moved C83 318.5 mm to (196.2, 118.0), turned to -90 degrees
- moved C75 317.8 mm to (192.2, 129.0)
- moved Y2 316.9 mm to (192.8, 118.0), turned to -90 degrees
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Connections:
- C63 pad 2: Net-(D114-A1) -> Net-(D115-A)
- D112 pad 1: Net-(D109-K) -> Net-(D110-K)
- D115 pad 2: Net-(D114-A1) -> Net-(D115-A)
- D116 pad 1: Net-(D114-A1) -> Net-(D115-A)
- D117 pad 1: Net-(D117-K) -> Net-(D114-A1)
- D117 pad 2: Net-(D114-A1) -> Net-(D115-A)
- FB4 pad 1: Net-(D159-K) -> Net-(Q6-D)
- J3 pad 1: /DIG_IN_GRP2/DIG_IN_TERMINAL_9 -> /DIG_IN_GRP2/COMC
- J3 pad 2: /DIG_IN_GRP2/DIG_IN_TERMINAL_8 -> /DIG_IN_GRP2/DIG_IN_TERMINAL_7
- J3 pad 3: /DIG_IN_GRP2/DIG_IN_TERMINAL_7 -> /DIG_IN_GRP2/DIG_IN_TERMINAL_8
- J3 pad 4: /DIG_IN_GRP2/COMC -> /DIG_IN_GRP2/DIG_IN_TERMINAL_9
- J34 pad 1: Net-(D117-K) -> Net-(D114-A1)
- J4 pad 1: Net-(D10-A1) -> Net-(D10-A2)
- J4 pad 2: Net-(D10-A2) -> Net-(D10-A1)
- J6 pad 1: /DIG_IN_GRP1/DIG_IN_TERMINAL_3 -> /DIG_IN_GRP1/COMA
- J6 pad 2: /DIG_IN_GRP1/DIG_IN_TERMINAL_2 -> /DIG_IN_GRP1/DIG_IN_TERMINAL_1
- J6 pad 3: /DIG_IN_GRP1/DIG_IN_TERMINAL_1 -> /DIG_IN_GRP1/DIG_IN_TERMINAL_2
- J6 pad 4: /DIG_IN_GRP1/COMA -> /DIG_IN_GRP1/DIG_IN_TERMINAL_3
- J7 pad 1: /DIG_IN_GRP1/DIG_IN_TERMINAL_6 -> /DIG_IN_GRP1/COMB
- J7 pad 2: /DIG_IN_GRP1/DIG_IN_TERMINAL_5 -> /DIG_IN_GRP1/DIG_IN_TERMINAL_4
- J7 pad 3: /DIG_IN_GRP1/DIG_IN_TERMINAL_4 -> /DIG_IN_GRP1/DIG_IN_TERMINAL_5
- J7 pad 4: /DIG_IN_GRP1/COMB -> /DIG_IN_GRP1/DIG_IN_TERMINAL_6
- J8 pad 1: /DIG_IN_GRP2/DIG_IN_TERMINAL_12 -> /DIG_IN_GRP2/COMD
- J8 pad 2: /DIG_IN_GRP2/DIG_IN_TERMINAL_11 -> /DIG_IN_GRP2/DIG_IN_TERMINAL_10
- J8 pad 3: /DIG_IN_GRP2/DIG_IN_TERMINAL_10 -> /DIG_IN_GRP2/DIG_IN_TERMINAL_11
- J8 pad 4: /DIG_IN_GRP2/COMD -> /DIG_IN_GRP2/DIG_IN_TERMINAL_12
- R184 pad 2: Net-(D114-A1) -> Net-(D115-A)
- R185 pad 1: Net-(D114-A1) -> Net-(D115-A)
Routing:
- net /ANALOG_OUT/AOUT2_V+: track 0.00 -> 28.9 mm, vias 0 -> 2
- net /ANALOG_OUT/AOUT1_V+: track 0.00 -> 28.9 mm, vias 0 -> 2
- net /ANALOG_OUT/AOUT1_V-: track 0.00 -> 27.1 mm, vias 0 -> 2
- net Net-(D109-K): track 0.00 -> 25.7 mm, vias 0 -> 2
- net Net-(D115-A): track 0.00 -> 25.7 mm, vias 0 -> 2
- net /ANALOG_OUT/AOUT2_V-: track 0.00 -> 24.2 mm, vias 0 -> 1
- net +3V3: track 122.2 -> 145.9 mm
- net Net-(U38-SET): track 0.00 -> 19.6 mm, vias 0 -> 2
- net Net-(U37-SET): track 0.00 -> 19.6 mm, vias 0 -> 2
- net Net-(D114-A2): track 0.00 -> 19.2 mm, vias 0 -> 2
- net Net-(D112-A2): track 0.00 -> 19.2 mm, vias 0 -> 2
- net Net-(J5-Pin_1): track 0.00 -> 17.6 mm
- net Net-(J40-Pin_1): track 0.00 -> 17.6 mm
- net Net-(U11-AVDD): track 0.00 -> 16.9 mm
- net Net-(D125-A1): track 0.00 -> 16.4 mm
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