File: Hardware/Running_Hardware/Open_STMPLC_IO_V0.1/ANALOG_IN.kicad_sch (KiCad schematic)
At the start: 67 parts, among them J35 Screw_Terminal_01x03, J36 Screw_Terminal_01x03, J37 Screw_Terminal_01x03, J38 Screw_Terminal_01x03, U39 AD4111, U40 REF3025, Y2 16MHz

Commit message: Gerber generation v0.1
Other:
- company: (none) -> Thingslista Automation LLP
Changed lines of the file:
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@@
 	(title_block
 		(title "Open_STMPLC_IO")
-		(date "2026-05-23")
+		(date "2026-06-03")
 		(rev "0.1")
+		(company "Thingslista Automation LLP")
 	)
 	(rectangle
