File: Hardware/Running_Hardware/Open_STMPLC_IO_V0.1/DIG_HS_OUT_4.kicad_sch (KiCad schematic)
At the start: 25 parts, among them Q4 2N7002K, U18 TPS26600PWP, U19 NVTFS5124PLTAG

Commit message: Gerber generation v0.1
Other:
- company: (none) -> Thingslista Automation LLP
Changed lines of the file:
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@@
 	(title_block
 		(title "Open_STMPLC_IO")
-		(date "2026-05-23")
+		(date "2026-06-03")
 		(rev "0.1")
+		(company "Thingslista Automation LLP")
 	)
 	(rectangle
