File: Hardware/Running_Hardware/Open_STMPLC_Main_V0.1/Open_STMPLC_Main_V0.1.kicad_pcb (KiCad board)
At the start: 2 copper layers, 168.8 x 90 mm, 129 parts, among them J1 Conn_02x08_Odd_Even, J10 10144518-041802LF, J11 HY951180A, J2 USB C, J3 TF-102, J5 Conn_Coaxial, J6 Conn_Coaxial, J7 Simcard_Nano, J8 10144518-041802LF, J9 10144518-041802LF, Q1 DTC143Z, Q2 DTC143Z, Q3 DTC143Z, Q4 DTC143Z, Q5 DTC143Z, Q6 DTC143Z, Q7 DTC143Z, SW1 Switch, SW2 SW_SPDT, SW3 Switch_6x6, U1 STM32F407ZGTx, U2 ADM2587E, U3 TPS3430WDRC, U4 CH340C, U5 TPD4E1U06DCKR, U6 W25Q64JVSSIQ, U7 LAN8720A, U8 EC200U, Y1 48MHz, Y2 32.768kHz

Commit message: IO board layout
Parts:
- moved U1 178.0 mm to (158.6, 115.0)
- moved C21 171.9 mm to (192.7, 56.0)
- moved C23 171.9 mm to (192.7, 58.5)
- moved C24 171.9 mm to (192.7, 61.0)
- moved C26 171.9 mm to (192.7, 63.5)
- moved R1 171.9 mm to (197.1, 58.5)
- moved R2 171.9 mm to (197.1, 61.0)
- moved R3 171.9 mm to (197.1, 63.5)
- moved C1 171.9 mm to (184.0, 56.0)
- moved C10 171.9 mm to (184.0, 68.5)
- moved C11 171.9 mm to (184.0, 71.0)
- moved C12 171.9 mm to (188.4, 56.0)
- moved C13 171.9 mm to (188.4, 58.5)
- moved C14 171.9 mm to (188.4, 61.0)
- moved C16 171.9 mm to (188.4, 63.5)
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
Commit message: Main PCB component placement
Parts:
- removed J3: TF-102, Connector_Card:microSD_HC_Molex_47219-2001
- removed R14, R15, R16, R17: 10K, Resistor_SMD:R_0603_1608Metric_Pad0.98x0.95mm_HandSolder
- added C55: 22uF, Capacitor_SMD:C_0805_2012Metric_Pad1.18x1.45mm_HandSolder, F.Cu at (66.5, 132.5)
- added C56: 22uF, Capacitor_SMD:C_0805_2012Metric_Pad1.18x1.45mm_HandSolder, F.Cu at (66.5, 135.0)
- added C57: 10pF, Capacitor_SMD:C_0603_1608Metric_Pad1.08x0.95mm_HandSolder, F.Cu at (215.0, 69.5)
- added C58: 10pF, Capacitor_SMD:C_0603_1608Metric_Pad1.08x0.95mm_HandSolder, F.Cu at (215.0, 78.5)
- added C59: 100nF, Capacitor_SMD:C_0603_1608Metric_Pad1.08x0.95mm_HandSolder, F.Cu at (158.5, 80.5)
- added C60: 100nF, Capacitor_SMD:C_0603_1608Metric_Pad1.08x0.95mm_HandSolder, F.Cu at (152.0, 80.5)
- added C61: 2.2uF, Capacitor_SMD:C_0603_1608Metric_Pad1.08x0.95mm_HandSolder, F.Cu at (177.0, 90.0)
- added C62: 2.2uF, Capacitor_SMD:C_0603_1608Metric_Pad1.08x0.95mm_HandSolder, F.Cu at (167.0, 112.5)
- added C63: 100nF, Capacitor_SMD:C_0603_1608Metric_Pad1.08x0.95mm_HandSolder, F.Cu at (145.0, 106.0)
- added C64: 1uF, Capacitor_SMD:C_0603_1608Metric_Pad1.08x0.95mm_HandSolder, F.Cu at (143.0, 106.0)
- added C79: 10uF, Capacitor_SMD:C_0805_2012Metric_Pad1.18x1.45mm_HandSolder, F.Cu at (176.5, 69.5)
- added C80: 100nF, Capacitor_SMD:C_0603_1608Metric_Pad1.08x0.95mm_HandSolder, F.Cu at (176.5, 67.0)
- added D6: DT1240A-08LP3810, Package_DFN_QFN:UDFN-9_1.0x3.8mm_P0.5mm, F.Cu at (176.5, 72.5)
- added J4: TF-01A, SD_Card_SideEntry:SD_Card, F.Cu at (174.5, 57.5)
- added L2: 3.3uH, Inductor_SMD:L_Abracon_ASPI-0630LR, F.Cu at (71.0, 126.5)
- added R67: 10K, Resistor_SMD:R_0603_1608Metric_Pad0.98x0.95mm_HandSolder, F.Cu at (183.5, 68.0)
- added R68: 10K, Resistor_SMD:R_0603_1608Metric_Pad0.98x0.95mm_HandSolder, F.Cu at (181.5, 68.0)
- added R69: 10K, Resistor_SMD:R_0603_1608Metric_Pad0.98x0.95mm_HandSolder, F.Cu at (179.5, 68.0)
- added R70: 10K, Resistor_SMD:R_0603_1608Metric_Pad0.98x0.95mm_HandSolder, F.Cu at (173.5, 68.5)
- added R71: 10K, Resistor_SMD:R_0603_1608Metric_Pad0.98x0.95mm_HandSolder, F.Cu at (171.5, 68.5)
- added R72: 10K, Resistor_SMD:R_0603_1608Metric_Pad0.98x0.95mm_HandSolder, F.Cu at (169.5, 68.5)
- added R73: 10K, Resistor_SMD:R_0603_1608Metric_Pad0.98x0.95mm_HandSolder, F.Cu at (167.5, 68.5)
- added TP5: TestPoint, TestPoint:TestPoint_Pad_D1.5mm, F.Cu at (70.0, 134.0)
- added Y3: 25MHz, Crystal:Crystal_SMD_5032-4Pin_5.0x3.2mm, F.Cu at (214.5, 74.0)
- SW1: footprint Button_Switch_SMD:SW_SPST_PTS810 -> Button_Switch_THT:SW_PUSH_6mm_H5mm
- U1: value STM32F407ZGTx -> STM32F407IGTx; footprint Package_QFP:LQFP-144_20x20mm_P0.5mm -> Package_QFP:LQFP-176_24x24mm_P0.5mm
- U5: value TPD4E1U06DCKR -> AP63203WU; footprint Package_TO_SOT_SMD:SOT-363_SC-70-6 -> Package_TO_SOT_SMD:TSOT-23-6
- moved BT1 82.1 mm to (136.4, 125.5), turned to 180 degrees
- moved R1 76.9 mm to (137.2, 106.8), turned to -90 degrees
- moved D1 74.3 mm to (137.4, 120.8), turned to 180 degrees
- moved U5 73.8 mm to (62.0, 127.5)
- moved SW1 70.4 mm to (127.8, 102.8)
- moved C32 69.4 mm to (62.0, 131.0)
- moved C1 67.7 mm to (139.2, 106.8), turned to 90 degrees
- moved R3 65.6 mm to (138.5, 93.0)
- moved R20 63.8 mm to (167.9, 130.4), turned to 90 degrees
- moved C12 63.3 mm to (158.0, 111.5), turned to 180 degrees
- moved C3 61.2 mm to (140.0, 103.5), turned to 180 degrees
- moved C34 60.2 mm to (164.4, 127.4), turned to 180 degrees
- moved C13 58.8 mm to (163.0, 111.5), turned to 180 degrees
- moved C2 57.5 mm to (140.0, 95.5)
- moved C33 54.0 mm to (66.0, 127.0), turned to 90 degrees
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Connections:
- C10 pad 1: Net-(U1-VDDA) -> /Microcontroller/3V3_MCU
- C11 pad 1: Net-(U1-VDDA) -> /Microcontroller/3V3_MCU
- C12 pad 1: Net-(U1-VDDA) -> /Microcontroller/3V3_MCU
- C13 pad 1: Net-(U1-VDDA) -> /Microcontroller/3V3_MCU
- C14 pad 1: Net-(U1-VDDA) -> /Microcontroller/3V3_MCU
- C15 pad 1: /MODBUS/3V3_ISO -> /B2B_Connector/3V3_ISO
- C16 pad 1: Net-(U1-VDDA) -> /Microcontroller/3V3_MCU
- C17 pad 1: /MODBUS/3V3_ISO -> /B2B_Connector/3V3_ISO
- C18 pad 1: Net-(U1-VDDA) -> /Microcontroller/3V3_MCU
- C21 pad 1: Net-(U1-VDDA) -> /Microcontroller/3V3_MCU
- C22 pad 1: /MODBUS/3V3_ISO -> /B2B_Connector/3V3_ISO
- C23 pad 1: Net-(U1-VDDA) -> /Microcontroller/3V3_MCU
- C24 pad 1: Net-(U1-VDDA) -> /Microcontroller/3V3_MCU
- C25 pad 1: /MODBUS/3V3_ISO -> /B2B_Connector/3V3_ISO
- C26 pad 1: Net-(U1-VDDA) -> /Microcontroller/3V3_MCU
- C27 pad 1: Net-(U1-VDDA) -> /Microcontroller/3V3_MCU
- C32 pad 1: +3V3 -> +24V
- C33 pad 1: +3V3 -> Net-(U5-SW)
- C33 pad 2: GND -> Net-(U5-BST)
- C8 pad 1: Net-(U1-VDDA) -> /Microcontroller/3V3_MCU
- C9 pad 1: Net-(U1-VDDA) -> /Microcontroller/3V3_MCU
- J1 pad 2: unconnected-(J1-Pin_2-Pad2) -> +3V3
- J10 pad 1: unconnected-(J10-Pin_1-Pad1) -> GND
- J10 pad 10: unconnected-(J10-Pin_10-Pad10) -> /B2B_Connector/DIG_OUT_~{FAULT}_5
- J10 pad 11: unconnected-(J10-Pin_11-Pad11) -> /B2B_Connector/DIG_OUT_DIAG_6
- J10 pad 12: unconnected-(J10-Pin_12-Pad12) -> /B2B_Connector/DIG_OUT_DIAG_5
- J10 pad 13: unconnected-(J10-Pin_13-Pad13) -> /B2B_Connector/DIG_OUT_6
- J10 pad 14: unconnected-(J10-Pin_14-Pad14) -> /B2B_Connector/DIG_OUT_5
- J10 pad 15: unconnected-(J10-Pin_15-Pad15) -> /B2B_Connector/RUN_LED
- J10 pad 16: unconnected-(J10-Pin_16-Pad16) -> /B2B_Connector/FAULT_LED
- J10 pad 17: unconnected-(J10-Pin_17-Pad17) -> /B2B_Connector/DIG_OUT_~{FAULT}_4
- J10 pad 18: unconnected-(J10-Pin_18-Pad18) -> /B2B_Connector/DIG_OUT_~{FAULT}_3
- J10 pad 19: unconnected-(J10-Pin_19-Pad19) -> /B2B_Connector/DIG_OUT_DIAG_4
- J10 pad 2: unconnected-(J10-Pin_2-Pad2) -> GND
- J10 pad 20: unconnected-(J10-Pin_20-Pad20) -> /B2B_Connector/DIG_OUT_DIAG_3
- J10 pad 21: unconnected-(J10-Pin_21-Pad21) -> /B2B_Connector/DIG_OUT_4
- J10 pad 22: unconnected-(J10-Pin_22-Pad22) -> /B2B_Connector/DIG_OUT_3
- J10 pad 23: unconnected-(J10-Pin_23-Pad23) -> /B2B_Connector/DIG_OUT_2
- J10 pad 24: unconnected-(J10-Pin_24-Pad24) -> /B2B_Connector/DIG_OUT_1
- J10 pad 25: unconnected-(J10-Pin_25-Pad25) -> /B2B_Connector/DIG_OUT_DIAG_2
- J10 pad 26: unconnected-(J10-Pin_26-Pad26) -> /B2B_Connector/DIG_OUT_DIAG_1
- J10 pad 27: unconnected-(J10-Pin_27-Pad27) -> /B2B_Connector/DIG_OUT_~{FAULT}_2
- J10 pad 28: unconnected-(J10-Pin_28-Pad28) -> /B2B_Connector/DIG_OUT_~{FAULT}_1
- J10 pad 29: unconnected-(J10-Pin_29-Pad29) -> /B2B_Connector/3V3_ISO
- J10 pad 3: unconnected-(J10-Pin_3-Pad3) -> /B2B_Connector/DIG_OUT_~{FAULT}_7
- J10 pad 30: unconnected-(J10-Pin_30-Pad30) -> GND
- J10 pad 31: unconnected-(J10-Pin_31-Pad31) -> GND_MODBUS
- J10 pad 32: unconnected-(J10-Pin_32-Pad32) -> GND_MODBUS
- J10 pad 33: unconnected-(J10-Pin_33-Pad33) -> /B2B_Connector/YZ-
- J10 pad 34: unconnected-(J10-Pin_34-Pad34) -> /B2B_Connector/AB-
- J10 pad 35: unconnected-(J10-Pin_35-Pad35) -> /B2B_Connector/YZ+
- J10 pad 36: unconnected-(J10-Pin_36-Pad36) -> /B2B_Connector/AB+
- J10 pad 37: unconnected-(J10-Pin_37-Pad37) -> GND_MODBUS
- J10 pad 38: unconnected-(J10-Pin_38-Pad38) -> GND_MODBUS
- J10 pad 39: unconnected-(J10-Pin_39-Pad39) -> GND
- J10 pad 4: unconnected-(J10-Pin_4-Pad4) -> /B2B_Connector/DIG_OUT_~{FAULT}_8
- J10 pad 40: unconnected-(J10-Pin_40-Pad40) -> GND
- J10 pad 5: unconnected-(J10-Pin_5-Pad5) -> /B2B_Connector/DIG_OUT_DIAG_7
- J10 pad 6: unconnected-(J10-Pin_6-Pad6) -> /B2B_Connector/DIG_OUT_DIAG_8
- J10 pad 7: unconnected-(J10-Pin_7-Pad7) -> /B2B_Connector/DIG_OUT_7
- J10 pad 8: unconnected-(J10-Pin_8-Pad8) -> /B2B_Connector/DIG_OUT_8
- J10 pad 9: unconnected-(J10-Pin_9-Pad9) -> /B2B_Connector/DIG_OUT_~{FAULT}_6
- J8 pad 1: unconnected-(J8-Pin_1-Pad1) -> GND
- J8 pad 10: unconnected-(J8-Pin_10-Pad10) -> /B2B_Connector/AOUT_~{OD}_2
- J8 pad 11: unconnected-(J8-Pin_11-Pad11) -> /B2B_Connector/AOUT_EFOT_1
- J8 pad 12: unconnected-(J8-Pin_12-Pad12) -> /B2B_Connector/AOUT_EFOT_2
- J8 pad 13: unconnected-(J8-Pin_13-Pad13) -> /B2B_Connector/AOUT_EFLD_1
- J8 pad 14: unconnected-(J8-Pin_14-Pad14) -> /B2B_Connector/AOUT_EFLD_2
- J8 pad 15: unconnected-(J8-Pin_15-Pad15) -> /B2B_Connector/AOUT_EFCM_1
- J8 pad 16: unconnected-(J8-Pin_16-Pad16) -> /B2B_Connector/AOUT_EFCM_2
- J8 pad 17: unconnected-(J8-Pin_17-Pad17) -> /B2B_Connector/TEMP_MISO
- J8 pad 18: unconnected-(J8-Pin_18-Pad18) -> /B2B_Connector/THRM_~{CS}
- J8 pad 19: unconnected-(J8-Pin_19-Pad19) -> /B2B_Connector/RTD_~{CS}_1
- J8 pad 2: unconnected-(J8-Pin_2-Pad2) -> GND
- J8 pad 20: unconnected-(J8-Pin_20-Pad20) -> /B2B_Connector/THRM_~{FAULT}
- J8 pad 21: unconnected-(J8-Pin_21-Pad21) -> /B2B_Connector/RTD_~{CS}_2
- J8 pad 22: unconnected-(J8-Pin_22-Pad22) -> /B2B_Connector/RTD_~{DRDY}_1
- J8 pad 23: unconnected-(J8-Pin_23-Pad23) -> /B2B_Connector/TEMP_SCLK
- J8 pad 24: unconnected-(J8-Pin_24-Pad24) -> /B2B_Connector/THRM_~{DRDY}
- J8 pad 25: unconnected-(J8-Pin_25-Pad25) -> /B2B_Connector/TEMP_MOSI
- J8 pad 26: unconnected-(J8-Pin_26-Pad26) -> /B2B_Connector/RTD_~{DRDY}_2
- J8 pad 27: unconnected-(J8-Pin_27-Pad27) -> /B2B_Connector/DIG_IN_6
- J8 pad 28: unconnected-(J8-Pin_28-Pad28) -> /GSM_STATUS_LED
- J8 pad 29: unconnected-(J8-Pin_29-Pad29) -> /B2B_Connector/DIG_IN_5
- J8 pad 3: unconnected-(J8-Pin_3-Pad3) -> /B2B_Connector/AOUT_VIN_1
- J8 pad 30: unconnected-(J8-Pin_30-Pad30) -> /NET_MODE_LED
- J8 pad 31: unconnected-(J8-Pin_31-Pad31) -> /B2B_Connector/DIG_IN_4
- J8 pad 32: unconnected-(J8-Pin_32-Pad32) -> /NET_STATUS_LED
- J8 pad 33: unconnected-(J8-Pin_33-Pad33) -> /B2B_Connector/DIG_IN_3
- J8 pad 35: unconnected-(J8-Pin_35-Pad35) -> /B2B_Connector/DIG_IN_2
- J8 pad 37: unconnected-(J8-Pin_37-Pad37) -> /B2B_Connector/DIG_IN_1
- J8 pad 39: unconnected-(J8-Pin_39-Pad39) -> GND
- J8 pad 4: unconnected-(J8-Pin_4-Pad4) -> /B2B_Connector/AOUT_VIN_2
- J8 pad 40: unconnected-(J8-Pin_40-Pad40) -> GND
- J8 pad 5: unconnected-(J8-Pin_5-Pad5) -> /B2B_Connector/AOUT_M1_1
- J8 pad 6: unconnected-(J8-Pin_6-Pad6) -> /B2B_Connector/AOUT_M1_2
- J8 pad 7: unconnected-(J8-Pin_7-Pad7) -> /B2B_Connector/AOUT_M2_1
- J8 pad 8: unconnected-(J8-Pin_8-Pad8) -> /B2B_Connector/AOUT_M2_2
- J8 pad 9: unconnected-(J8-Pin_9-Pad9) -> /B2B_Connector/AOUT_~{OD}_1
- J9 pad 1: unconnected-(J9-Pin_1-Pad1) -> GND
- J9 pad 10: unconnected-(J9-Pin_10-Pad10) -> /B2B_Connector/DIG_HS_IMON_2
- J9 pad 11: unconnected-(J9-Pin_11-Pad11) -> /B2B_Connector/DIG_HS_~{FAULT}_1
- J9 pad 12: unconnected-(J9-Pin_12-Pad12) -> /B2B_Connector/DIG_HS_~{FAULT}_2
- J9 pad 13: unconnected-(J9-Pin_13-Pad13) -> /B2B_Connector/DIG_HS_OUT_1
- J9 pad 14: unconnected-(J9-Pin_14-Pad14) -> /B2B_Connector/DIG_HS_OUT_2
- J9 pad 15: unconnected-(J9-Pin_15-Pad15) -> GND
- J9 pad 16: unconnected-(J9-Pin_16-Pad16) -> GND
- J9 pad 17: unconnected-(J9-Pin_17-Pad17) -> /B2B_Connector/DIG_HS_OUT_3
- J9 pad 18: unconnected-(J9-Pin_18-Pad18) -> /B2B_Connector/DIG_HS_OUT_4
- J9 pad 19: unconnected-(J9-Pin_19-Pad19) -> /B2B_Connector/DIG_HS_~{SHDN}_3
- J9 pad 2: unconnected-(J9-Pin_2-Pad2) -> GND
- J9 pad 20: unconnected-(J9-Pin_20-Pad20) -> /B2B_Connector/DIG_HS_~{SHDN}_4
- J9 pad 21: unconnected-(J9-Pin_21-Pad21) -> /B2B_Connector/DIG_HS_~{FAULT}_3
- J9 pad 22: unconnected-(J9-Pin_22-Pad22) -> /B2B_Connector/DIG_HS_IMON_4
- J9 pad 23: unconnected-(J9-Pin_23-Pad23) -> /B2B_Connector/DIG_HS_IMON_3
- J9 pad 24: unconnected-(J9-Pin_24-Pad24) -> /B2B_Connector/DIG_HS_~{FAULT}_4
- J9 pad 25: unconnected-(J9-Pin_25-Pad25) -> GND
- J9 pad 26: unconnected-(J9-Pin_26-Pad26) -> GND
- J9 pad 27: unconnected-(J9-Pin_27-Pad27) -> /B2B_Connector/ANALOG_IN_DOUT
- J9 pad 28: unconnected-(J9-Pin_28-Pad28) -> /B2B_Connector/ANALOG_IN_CS
- J9 pad 29: unconnected-(J9-Pin_29-Pad29) -> /B2B_Connector/ANALOG_IN_DIN
- J9 pad 3: unconnected-(J9-Pin_3-Pad3) -> +24V
- J9 pad 30: unconnected-(J9-Pin_30-Pad30) -> /B2B_Connector/ANALOG_IN_ERROR
- J9 pad 31: unconnected-(J9-Pin_31-Pad31) -> /B2B_Connector/ANALOG_IN_SCLK
- J9 pad 32: unconnected-(J9-Pin_32-Pad32) -> GND
- J9 pad 33: unconnected-(J9-Pin_33-Pad33) -> /B2B_Connector/DIG_IN_10
- J9 pad 34: unconnected-(J9-Pin_34-Pad34) -> /B2B_Connector/DIG_IN_7
- J9 pad 35: unconnected-(J9-Pin_35-Pad35) -> /B2B_Connector/DIG_IN_11
- J9 pad 36: unconnected-(J9-Pin_36-Pad36) -> /B2B_Connector/DIG_IN_8
- J9 pad 37: unconnected-(J9-Pin_37-Pad37) -> /B2B_Connector/DIG_IN_12
- J9 pad 38: unconnected-(J9-Pin_38-Pad38) -> /B2B_Connector/DIG_IN_9
- J9 pad 39: unconnected-(J9-Pin_39-Pad39) -> GND
- J9 pad 4: unconnected-(J9-Pin_4-Pad4) -> +3V3
- J9 pad 40: unconnected-(J9-Pin_40-Pad40) -> GND
- J9 pad 5: unconnected-(J9-Pin_5-Pad5) -> +24V
- J9 pad 6: unconnected-(J9-Pin_6-Pad6) -> +3V3
- J9 pad 7: unconnected-(J9-Pin_7-Pad7) -> /B2B_Connector/DIG_HS_~{SHDN}_1
- J9 pad 8: unconnected-(J9-Pin_8-Pad8) -> /B2B_Connector/DIG_HS_~{SHDN}_2
- J9 pad 9: unconnected-(J9-Pin_9-Pad9) -> /B2B_Connector/DIG_HS_IMON_1
- Q1 pad 3: /GSM_Module/NET_STATUS_LED -> /NET_STATUS_LED
- Q3 pad 3: /GSM_Module/NET_MODE_LED -> /NET_MODE_LED
- Q5 pad 3: /GSM_Module/STATUS_LED -> /GSM_STATUS_LED
- R1 pad 1: Net-(U1-VDDA) -> /Microcontroller/3V3_MCU
- R3 pad 2: Net-(U1-VDDA) -> /Microcontroller/3V3_MCU
- U1 pad 10: unconnected-(U1-PF0-Pad10) -> Net-(U1-PC15)
- U1 pad 102: unconnected-(U1-PA10-Pad102) -> GND
- U1 pad 103: unconnected-(U1-PA11-Pad103) -> /Microcontroller/3V3_MCU
- U1 pad 107: GND -> unconnected-(U1-PG3-Pad107)
- U1 pad 108: Net-(U1-VDDA) -> unconnected-(U1-PG4-Pad108)
- U1 pad 113: unconnected-(U1-PC12-Pad113) -> GND
- U1 pad 114: unconnected-(U1-PD0-Pad114) -> /Microcontroller/3V3_MCU
- U1 pad 120: GND -> unconnected-(U1-PA9-Pad120)
- U1 pad 121: Net-(U1-VDDA) -> unconnected-(U1-PA10-Pad121)
- U1 pad 125: unconnected-(U1-PG10-Pad125) -> Net-(U1-VCAP_2)
- U1 pad 126: unconnected-(U1-PG11-Pad126) -> GND
- U1 pad 127: unconnected-(U1-PG12-Pad127) -> /Microcontroller/3V3_MCU
- U1 pad 130: GND -> unconnected-(U1-PH15-Pad130)
- U1 pad 131: Net-(U1-VDDA) -> unconnected-(U1-PI0-Pad131)
- U1 pad 135: unconnected-(U1-PB5-Pad135) -> GND
- U1 pad 136: unconnected-(U1-PB6-Pad136) -> /Microcontroller/3V3_MCU
- U1 pad 138: Net-(U1-BOOT0) -> unconnected-(U1-PA15-Pad138)
- U1 pad 14: unconnected-(U1-PF4-Pad14) -> GND
- U1 pad 144: Net-(U1-VDDA) -> unconnected-(U1-PD2-Pad144)
- U1 pad 15: unconnected-(U1-PF5-Pad15) -> /Microcontroller/3V3_MCU
- U1 pad 16: GND -> unconnected-(U1-PF0-Pad16)
- U1 pad 17: Net-(U1-VDDA) -> unconnected-(U1-PF1-Pad17)
- U1 pad 22: unconnected-(U1-PF10-Pad22) -> GND
- U1 pad 23: Net-(U1-PH0) -> /Microcontroller/3V3_MCU
- U1 pad 24: Net-(U1-PH1) -> unconnected-(U1-PF6-Pad24)
- U1 pad 25: /Microcontroller/~{WDO} -> unconnected-(U1-PF7-Pad25)
- U1 pad 29: unconnected-(U1-PC3-Pad29) -> Net-(U1-PH0)
- U1 pad 30: Net-(U1-VDDA) -> Net-(U1-PH1)
- U1 pad 31: GND -> /Microcontroller/~{WDO}
- U1 pad 33: Net-(U1-VDDA) -> unconnected-(U1-PC1-Pad33)
- U1 pad 36: unconnected-(U1-PA2-Pad36) -> /Microcontroller/3V3_MCU
- U1 pad 37: unconnected-(U1-PA3-Pad37) -> GND
- U1 pad 38: GND -> /Microcontroller/3V3_MCU
- U1 pad 39: Net-(U1-VDDA) -> /Microcontroller/3V3_MCU
- U1 pad 49: unconnected-(U1-PF11-Pad49) -> /Microcontroller/3V3_MCU
- U1 pad 51: GND -> unconnected-(U1-PA5-Pad51)
- U1 pad 52: Net-(U1-VDDA) -> unconnected-(U1-PA6-Pad52)
- U1 pad 62: Net-(U1-VDDA) -> /Microcontroller/3V3_MCU
- U1 pad 71: unconnected-(U1-VCAP_1-Pad71) -> GND
- U1 pad 72: Net-(U1-VDDA) -> /Microcontroller/3V3_MCU
- U1 pad 8: Net-(U1-PC14) -> unconnected-(U1-PC13-Pad8)
- U1 pad 81: unconnected-(U1-PD12-Pad81) -> Net-(U1-VCAP_1)
- U1 pad 82: unconnected-(U1-PD13-Pad82) -> /Microcontroller/3V3_MCU
- U1 pad 83: GND -> unconnected-(U1-PH6-Pad83)
- U1 pad 84: Net-(U1-VDDA) -> unconnected-(U1-PH7-Pad84)
- U1 pad 9: Net-(U1-PC15) -> Net-(U1-PC14)
- U1 pad 90: unconnected-(U1-PG5-Pad90) -> GND
- U1 pad 91: unconnected-(U1-PG6-Pad91) -> /Microcontroller/3V3_MCU
- U1 pad 94: GND -> unconnected-(U1-PB14-Pad94)
- U1 pad 95: Net-(U1-VDDA) -> unconnected-(U1-PB15-Pad95)
- U2 pad 12: /MODBUS/3V3_ISO -> /B2B_Connector/3V3_ISO
- U2 pad 13: /MODBUS/Y -> /B2B_Connector/YZ+
- U2 pad 15: /MODBUS/Z -> /B2B_Connector/YZ-
- U2 pad 17: /MODBUS/B -> /B2B_Connector/AB+
- U2 pad 18: /MODBUS/A -> /B2B_Connector/AB-
- U2 pad 19: /MODBUS/3V3_ISO -> /B2B_Connector/3V3_ISO
- U5 pad 1: /Storage/SD_MISO -> +3V3
- U5 pad 2: GND -> +24V
- U5 pad 3: /Storage/SD_CS -> +24V
- U5 pad 4: /Storage/SD_MOSI -> GND
- U5 pad 5: unconnected-(U5-NC-Pad5) -> Net-(U5-SW)
- U5 pad 6: /Storage/SD_CLK -> Net-(U5-BST)
- U6 pad 2: /Storage/SD_MISO -> /Microcontroller/SD_MISO
- U6 pad 5: /Storage/SD_MOSI -> /Microcontroller/SD_MOSI
- U7 pad 4: unconnected-(U7-XTAL2-Pad4) -> Net-(U7-XTAL2)
- U7 pad 5: unconnected-(U7-XTAL1/CLKIN-Pad5) -> Net-(U7-XTAL1/CLKIN)
