File: Hardware/Running_Hardware/Open_STMPLC_Main_V0.1/Storage.kicad_sch (KiCad schematic)
At the start: 14 parts, among them J5 TF-102, U5 W25Q64JVSSIQ, U6 TPD4E1U06DCKR

Commit message: Main PCB schematic changes V0.1
Other:
- title: (none) -> Open_STMPLC_Main
Changed lines of the file:
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@@
 	(generator_version "9.0")
 	(paper "A4")
+	(title_block
+		(title "Open_STMPLC_Main")
+		(date "2026-04-04")
+		(rev "0.1")
+	)
 	(rectangle
 		(start 166.37 15.24)

Commit message: Pin mapping IO connector
Parts:
- added D6: DT1240A-08LP3810, Package_DFN_QFN:UDFN-9_1.0x3.8mm_P0.5mm, symbol Power_Protection:DT1240A-08LP3810
- added J4: TF-01A, SD_Card_SideEntry:SD_Card, symbol Connector:Micro_SD_Card_Det1
- added R67, R68, R69, R70, R71, R72, R73: 10K, Resistor_SMD:R_0603_1608Metric_Pad0.98x0.95mm_HandSolder, symbol Device:R_Small
- U5: renamed from U6; footprint Package_TO_SOT_SMD:SOT-363_SC-70-6_Handsoldering -> Package_TO_SOT_SMD:SOT-363_SC-70-6
- renumbered C32 to C34, C33 to C35, C24 to C79, C25 to C80, J5 to J3, R110 to R14, R111 to R15, R112 to R16, R28 to R17, R113 to R18, R109 to R19, R114 to R20, U5 to U6
Connections:
- net +3V3: now also J4.4 (VDD), R67.1, R68.1, R69.1, R70.1, R71.1, R72.1, R73.1
- net GND: now also D6.3 (A), J4.10 (SHIELD), J4.6 (VSS)
- net SD_CLK: now also D6.8 (K7), J4.5 (CLK), R70.2
- new net +3V3_PERI: D6.7 (K6)
- new net SD_CMD: D6.4 (K3), J4.3 (CMD), R71.2
- new net SD_DAT0: D6.2 (K2), J4.7 (DAT0), R69.2
- new net SD_DAT1: D6.1 (K1), J4.8 (DAT1), R68.2
- new net SD_DAT2: D6.6 (K5), J4.1 (DAT2), R73.2
- new net SD_DAT3: D6.5 (K4), J4.2 (DAT3/CD), R72.2
- new net SD_DET: D6.9 (K8), J4.9 (DET), R67.2

Commit message: IO board layout
Parts:
- removed J3: TF-102, Connector_Card:microSD_HC_Molex_47219-2001, symbol Connector:Micro_SD_Card
- removed R14, R15, R16, R17: 10K, Resistor_SMD:R_0603_1608Metric_Pad0.98x0.95mm_HandSolder, symbol Device:R_Small
- removed U5: TPD4E1U06DCKR, Package_TO_SOT_SMD:SOT-363_SC-70-6, symbol TVS_Diode:TPD4E1U06DCKR
Connections:
- net +3V3_PERI is gone; now on net +3V3: D6.7 (K6)
- no-connect marks 2 -> 0
Other:
- moved on the sheet: D6, J4, R67, R68, R69, R70, R71, R72, R73

Commit message: Component placement main pcb
Connections:
- net SD_CLK: no longer U6.6 (CLK)
- net SD_MISO renamed Flash_MISO
- net SD_MOSI renamed Flash_MOSI
- new net Flash_CLK: U6.6 (CLK)
Changed lines of the file:
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@@
 	(wire
 		(pts
-			(xy 48.26 87.63) (xy 59.69 87.63)
+			(xy 55.88 87.63) (xy 59.69 87.63)
 		)
 		(stroke
@@
 	(wire
 		(pts
-			(xy 48.26 67.31) (xy 82.55 67.31)
+			(xy 55.88 67.31) (xy 82.55 67.31)
 		)
 		(stroke
@@
 	(wire
 		(pts
-			(xy 48.26 80.01) (xy 67.31 80.01)
+			(xy 55.88 80.01) (xy 67.31 80.01)
 		)
 		(stroke
@@
 	(wire
 		(pts
-			(xy 48.26 82.55) (xy 63.5 82.55)
+			(xy 55.88 82.55) (xy 63.5 82.55)
 		)
 		(stroke
@@
 	(wire
 		(pts
-			(xy 48.26 69.85) (xy 78.74 69.85)
+			(xy 55.88 69.85) (xy 78.74 69.85)
 		)
 		(stroke
@@
 	(wire
 		(pts
-			(xy 48.26 64.77) (xy 86.36 64.77)
+			(xy 55.88 64.77) (xy 86.36 64.77)
 		)
 		(stroke
@@
 	(wire
 		(pts
-			(xy 48.26 74.93) (xy 71.12 74.93)
+			(xy 55.88 74.93) (xy 71.12 74.93)
 		)
 		(stroke
@@
 		)
 	)
-	(label "SD_CMD"
-		(at 48.26 69.85 0)
-		(effects
-			(font
-				(size 1 1)
-			)
-			(justify left bottom)
-		)
-	)
-	(label "SD_DET"
-		(at 48.26 87.63 0)
-		(effects
-			(font
-				(size 1 1)
-			)
-			(justify left bottom)
-		)
-	)
 	(label "SD_CLK"
 		(at 92.71 120.65 270)
@@
 		)
 	)
-	(label "SD_DAT1"
-		(at 48.26 82.55 0)
-		(effects
-			(font
-				(size 1 1)
-			)
-			(justify left bottom)
-		)
-	)
 	(label "SD_DET"
 		(at 95.25 120.65 270)
@@
 	)
 	(label "SD_DAT3"
-		(at 48.26 67.31 0)
-		(effects
-			(font
-				(size 1 1)
-			)
-			(justify left bottom)
-		)
-	)
-	(label "SD_DAT3"
 		(at 85.09 120.65 270)
 		(effects
@@
 		)
 	)
-	(label "SD_CLK"
-		(at 48.26 74.93 0)
-		(effects
-			(font
-				(size 1 1)
-			)
-			(justify left bottom)
-		)
-	)
-	(label "SD_DAT0"
-		(at 48.26 80.01 0)
-		(effects
-			(font
-				(size 1 1)
-			)
-			(justify left bottom)
-		)
-	)
 	(label "SD_DAT2"
 		(at 87.63 120.65 270)
@@
 		)
 	)
-	(label "SD_DAT2"
-		(at 48.26 64.77 0)
-		(effects
-			(font
-				(size 1 1)
-			)
-			(justify left bottom)
-		)
-	)
-	(hierarchical_label "SD_MISO"
+	(hierarchical_label "SD_DAT2"
+		(shape bidirectional)
+		(at 55.88 64.77 180)
+		(effects
+			(font
+				(size 1 1)
+			)
+			(justify right)
+		)
+	)
+	(hierarchical_label "SD_DAT3"
+		(shape bidirectional)
+		(at 55.88 67.31 180)
+		(effects
+			(font
+				(size 1 1)
+			)
+			(justify right)
+		)
+	)
+	(hierarchical_label "SD_CLK"
+		(shape input)
+		(at 55.88 74.93 180)
+		(effects
+			(font
+				(size 1 1)
+			)
+			(justify right)
+		)
+	)
+	(hierarchical_label "SD_CMD"
+		(shape input)
+		(at 55.88 69.85 180)
+		(effects
+			(font
+				(size 1 1)
+			)
+			(justify right)
+		)
+	)
+	(hierarchical_label "Flash_MISO"
 		(shape output)
 		(at 195.58 85.09 180)
@@
 		)
 	)
-	(hierarchical_label "SD_MOSI"
+	(hierarchical_label "Flash_MOSI"
 		(shape input)
 		(at 243.84 90.17 0)
@@
 		)
 	)
-	(hierarchical_label "SD_CLK"
+	(hierarchical_label "SD_DET"
+		(shape output)
+		(at 55.88 87.63 180)
+		(effects
+			(font
+				(size 1 1)
+			)
+			(justify right)
+		)
+	)
+	(hierarchical_label "Flash_CLK"
 		(shape input)
 		(at 243.84 87.63 0)
@@
 		)
 	)
+	(hierarchical_label "SD_DAT0"
+		(shape bidirectional)
+		(at 55.88 80.01 180)
+		(effects
+			(font
+				(size 1 1)
+			)
+			(justify right)
+		)
+	)
+	(hierarchical_label "SD_DAT1"
+		(shape bidirectional)
+		(at 55.88 82.55 180)
+		(effects
+			(font
+				(size 1 1)
+			)
+			(justify right)
+		)
+	)

Commit message: PCB routing completion v0.1 Main
Parts:
- removed D6: DT1240A-08LP3810, Package_DFN_QFN:UDFN-9_1.0x3.8mm_P0.5mm, symbol Power_Protection:DT1240A-08LP3810
- added D10, D11, D12, D13, D19, D5, D6, D9: UAD8C05L01, Diode_SMD:D_SOD-882, symbol Device:D_TVS_Small
Connections:
- net +3V3: now also D11.2 (A2)
- net GND: now also D10.1 (A1), D11.1 (A1), D12.1 (A1), D13.1 (A1), D19.1 (A1), D5.1 (A1), D6.1 (A1), D9.1 (A1)
- net SD_CLK: now also D12.2 (A2)
- net SD_CMD: now also D6.2 (A2)
- net SD_DAT0: now also D5.2 (A2)
- net SD_DAT1: now also D19.2 (A2)
- net SD_DAT2: now also D10.2 (A2)
- net SD_DAT3: now also D9.2 (A2)
- net SD_DET: now also D13.2 (A2)

Commit message: Gerber generation v0.1
Other:
- company: (none) -> Thingslista Automation LLP
Changed lines of the file:
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@@
 	(title_block
 		(title "Open_STMPLC_Main")
-		(date "2026-05-24")
+		(date "2026-06-03")
 		(rev "0.1")
+		(company "Thingslista Automation LLP")
 	)
 	(rectangle
